File: KiCad/Serverola-wiring/amplifier.kicad_sch (KiCad schematic)
At the start: 5 parts

Commit message: project renaming started with KiCad files
Parts:
- A1: symbol ProxVox-wiring:Headphone AMP 3 click -> Serverola-wiring:Headphone AMP 3 click
- A2: symbol ProxVox-wiring:USB To I2C Click -> Serverola-wiring:USB To I2C Click
- A3: symbol ProxVox-wiring:AudioAmp 8 Click -> Serverola-wiring:AudioAmp 8 Click
Connections:
- net at A1.10 (5V): now also A2.7 (+3.3V)
Changed lines of the file:
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@@
 		)
 		(instances
-			(project "ProxVox-wiring"
+			(project "Serverola-wiring"
 				(path "/b2d95b56-b830-46e8-8d1f-758749cc9f8d/2c7e2924-535e-40f3-8191-8c2c98bcddd8"
 					(reference "R2")
@@
 	)
 	(symbol
-		(lib_id "ProxVox-wiring:Headphone AMP 3 click")
+		(lib_id "Serverola-wiring:Headphone AMP 3 click")
 		(at 76.2 101.6 0)
 		(unit 1)
@@
 		)
 		(instances
-			(project "ProxVox-wiring"
+			(project "Serverola-wiring"
 				(path "/b2d95b56-b830-46e8-8d1f-758749cc9f8d/2c7e2924-535e-40f3-8191-8c2c98bcddd8"
 					(reference "A1")
@@
 		)
 		(instances
-			(project "ProxVox-wiring"
+			(project "Serverola-wiring"
 				(path "/b2d95b56-b830-46e8-8d1f-758749cc9f8d/2c7e2924-535e-40f3-8191-8c2c98bcddd8"
 					(reference "R1")
@@
 	)
 	(symbol
-		(lib_id "ProxVox-wiring:AudioAmp 8 Click")
+		(lib_id "Serverola-wiring:AudioAmp 8 Click")
 		(at 228.6 101.6 0)
 		(unit 1)
@@
 		)
 		(instances
-			(project "ProxVox-wiring"
+			(project "Serverola-wiring"
 				(path "/b2d95b56-b830-46e8-8d1f-758749cc9f8d/2c7e2924-535e-40f3-8191-8c2c98bcddd8"
 					(reference "A3")
@@
 	)
 	(symbol
-		(lib_id "ProxVox-wiring:USB To I2C Click")
+		(lib_id "Serverola-wiring:USB To I2C Click")
 		(at 152.4 101.6 0)
 		(unit 1)
@@
 		)
 		(instances
-			(project "ProxVox-wiring"
+			(project "Serverola-wiring"
 				(path "/b2d95b56-b830-46e8-8d1f-758749cc9f8d/2c7e2924-535e-40f3-8191-8c2c98bcddd8"
 					(reference "A2")
