File: KiCad/Serverola-wiring/power-button.kicad_sch (KiCad schematic)
At the start: 2 parts, among them SW1 Alps (original)

Commit message: project renaming started with KiCad files
Parts:
- P1: symbol ProxVox-wiring:IDC10_PLUG@10 -> Serverola-wiring:IDC10_PLUG@10
Changed lines of the file:
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@@
 		)
 		(instances
-			(project "ProxVox-wiring"
+			(project "Serverola-wiring"
 				(path "/b2d95b56-b830-46e8-8d1f-758749cc9f8d/dd736ac1-64ad-4002-bc3e-8db70160fac5"
 					(reference "SW1")
@@
 	)
 	(symbol
-		(lib_id "ProxVox-wiring:IDC10_PLUG@10")
+		(lib_id "Serverola-wiring:IDC10_PLUG@10")
 		(at 43.18 48.26 0)
 		(unit 1)
@@
 		)
 		(instances
-			(project "ProxVox-wiring"
+			(project "Serverola-wiring"
 				(path "/b2d95b56-b830-46e8-8d1f-758749cc9f8d/dd736ac1-64ad-4002-bc3e-8db70160fac5"
 					(reference "P1")
